File: pcb/meowpad.kicad_sch (KiCad schematic)
At the start: 16 parts, among them J1 OLED_DISPLAY, SW1 SW_Push_45deg, SW2 SW_Push_45deg, SW3 SW_Push_45deg, SW4 SW_Push_45deg, SW6 SW_Push_45deg, U2 XIAO-RP2040-DIP

Commit message: bill of materials
Parts:
- U2: footprint Seeed Studio XIAO Series Library:XIAO-RA4M1-SMD -> Seeed Studio XIAO Series Library:XIAO-RP2040-DIP
Changed lines of the file:
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@@
 			)
 		)
-		(property "Footprint" "Seeed Studio XIAO Series Library:XIAO-RA4M1-SMD"
+		(property "Footprint" "Seeed Studio XIAO Series Library:XIAO-RP2040-DIP"
 			(at 66.548 65.278 0)
 			(effects
